File: MPL3115A2/MPL3115A2_barometer.sch (KiCad schematic (older format))
At the start: 4 parts, among them U1 MPL3115A2

Commit message: add test points to schematic (not layout). Add power signs in lower-right of schematic
Parts:
- added TP1: TestPoint, TestPoint:TestPoint_Keystone_5010-5014_Multipurpose, symbol Connector:TestPoint
- U1: symbol MPL3115A2_barometer-rescue:MPL3115A2-MPL3115A2 -> MPL3115A2_barometer-rescue:MPL3115A2-MPL3115A2-MPL3115A2_barometer-rescue
Connections:
- wire segments 21 -> 23
Changed lines of the file:
@@
 $EndComp
 Wire Wire Line
-	5850 3550 5500 3550
+	5850 3550 5600 3550
 Connection ~ 5500 3850
 Wire Wire Line
@@
 $EndComp
 $Comp
-L MPL3115A2_barometer-rescue:MPL3115A2-MPL3115A2 U1
+L MPL3115A2_barometer-rescue:MPL3115A2-MPL3115A2-MPL3115A2_barometer-rescue U1
 U 1 1 5F979C67
 P 6350 3750
@@
 Wire Wire Line
 	4350 3300 4600 3300
+$Comp
+L Connector:TestPoint TP1
+U 1 1 5FEA9553
+P 5600 2650
+F 0 "TP1" H 5658 2768 50  0000 L CNN
+F 1 "TestPoint" H 5658 2677 50  0000 L CNN
+F 2 "TestPoint:TestPoint_Keystone_5010-5014_Multipurpose" H 5800 2650 50  0001 C CNN
+F 3 "~" H 5800 2650 50  0001 C CNN
+	1    5600 2650
+	1    0    0    -1
+$EndComp
+Wire Wire Line
+	5600 2650 5600 3550
+Connection ~ 5600 3550
+Wire Wire Line
+	5600 3550 5500 3550
 $EndSCHEMATC
