File: hardware/rev1/_autosave-rev1.sch (KiCad schematic (older format))
At the start: 43 parts, among them J1 SD_socket, J2 Conn_01x08_Female, Q1 BSS138, Q2 BSS138, U1 74HC4050D,653, U1 MPL3115A2, U2 ASDMB-xxxMHz, U2 LP2985-3.3

Commit message: add level shifter to BNO055 schematic. Needs review
Parts:
- removed U?: DEV-14058, MODULE_DEV-14058, symbol teensy:DEV-14058
- J1: symbol formula:SD_socket -> rev1-rescue:SD_socket-formula
- U1: symbol formula:74HC4050D,653 -> rev1-rescue:74HC4050D,653-formula
- U?: symbol rocketry:MPL3115A2 -> rev1-rescue:MPL3115A2-rocketry
Other:
- moved on the sheet: C1, C2, C3, C4, C5, R1, R2, R3, R4, TP?, TP_GND
