File: hardware/rev1/_autosave-rev1.kicad_pcb (KiCad board)
At the start: 2 copper layers, 28 parts, among them U1 BNO055, U2 MPL3115A2, U3 Teensy3.6, Y1 Crystal_32kHz768

Commit message: wip
Parts:
- moved C8 33.3 mm to (151.5, 108.8), turned to 0 degrees
- moved C7 30.6 mm to (151.5, 110.8), turned to 0 degrees
- moved TP8 28.3 mm to (155.5, 114.5), turned to 0 degrees
- moved C9 28.0 mm to (151.5, 112.8), turned to 0 degrees
- moved U2 26.3 mm to (147.8, 113.0), turned to 0 degrees
- moved R3 24.6 mm to (134.5, 110.2)
- moved R4 24.6 mm to (131.2, 110.2)
- moved C1 24.6 mm to (135.4, 121.9)
- moved C2 24.6 mm to (135.4, 118.1)
- moved C3 24.6 mm to (135.4, 120.0)
- moved C5 24.6 mm to (138.0, 116.1)
- moved C6 24.6 mm to (138.0, 113.9)
- moved R2 24.6 mm to (131.0, 120.3)
- moved TP1 24.6 mm to (120.3, 107.5)
- moved TP2 24.6 mm to (124.0, 107.5)
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Routing:
- net COM3: track 5.18 -> 1.17 mm, vias 2 -> 1
- net SDA_TEENSY: track 5.03 -> 5.36 mm, vias 0 -> 1
- net SCL_TEENSY: track 5.12 -> 5.09 mm, vias 0 -> 1
