File: hardware/rev1/rev1.sch (KiCad schematic (older format))
At the start: 24 parts, among them J1 SD_socket, J2 Conn_01x08_Female, Q1 BSS138, Q2 BSS138, U1 74HC4050D,653, U1 MPL3115A2, U2 LP2985-3.3

Commit message: Try hierarchical schematic - second pass
Parts:
- removed U1: MPL3115A2, MPL3115A2_barometer:MPL3115A2, symbol MPL3115A2_barometer-rescue:MPL3115A2-MPL3115A2-MPL3115A2_barometer-rescue
- added C1, C4: 100nF, footprints:C_0805_OEM, symbol Device:C
- added C2: 6.8nF, footprints:C_0805_OEM, symbol Device:C
- added C3: 120nF, footprints:C_0805_OEM, symbol Device:C
- added C5: 0.01u, footprints:C_0603_1608Metric, symbol Device:C
- added J? (x2): Conn_02x03_Counter_Clockwise, symbol Connector_Generic:Conn_02x03_Counter_Clockwise
- added R1: Optional 10k, footprints:R_0805_OEM, symbol Device:R
- added R2: Pull-up 10k, footprints:R_0805_OEM, symbol Device:R
- added R3, R4: Rpull, footprints:R_0805_OEM, symbol Device:R
- added TP? (x4), TP_GND: TestPoint, symbol Connector:TestPoint
- added U2: ASDMB-xxxMHz, ASDK2-32.768KHZ-LR-T3:ASDK2-32.768KHZ-LR-T3, symbol Oscillator:ASDMB-xxxMHz
- added U?: MPL3115A2, symbol rocketry:MPL3115A2
- added U?: BNO055_BNO055, symbol bno055:BNO055_BNO055
Connections:
- net labels added: COM3, GNDIO, INT, INTERRUPT, OptionalOSCinput, OptionalOSCoutput, nBOOT_LOAD_PIN, nRESET
- wire segments 81 -> 194
- no-connect marks 2 -> 3
Other:
- moved on the sheet: C1, C2, C3, TP1

Commit message: Schematic: connect Teensy to BNO055 and MPL
Parts:
- removed C1, C3: 100nF, Capacitor_SMD:C_0805_2012Metric_Pad1.18x1.45mm_HandSolder, symbol Device:CP1
- removed C1, C3: C, symbol Device:C
- removed C2: 10uF, Capacitor_SMD:C_0805_2012Metric_Pad1.18x1.45mm_HandSolder, symbol Device:CP1
- removed C2: 0.1uF, symbol Device:CP1
- removed C3: 100n, footprints:C_0805_OEM, symbol Device:C
- removed D1: RED, symbol Device:LED
- removed J1: SD_socket, footprints:sd_socket_molex_5009980900, symbol formula:SD_socket
- removed J2: Conn_01x08_Female, symbol Connector:Conn_01x08_Female
- removed J? (x2): Conn_02x03_Counter_Clockwise, symbol Connector_Generic:Conn_02x03_Counter_Clockwise
- removed Q1, Q2: BSS138, Package_TO_SOT_SMD:SOT-23, symbol Transistor_FET:BSS138
- removed R1: 1_K, symbol Device:R
- removed R1, R2, R3, R4: R_10K, Resistor_SMD:R_0805_2012Metric_Pad1.20x1.40mm_HandSolder, symbol Device:R
- removed U1: 74HC4050D,653, SOIC127P600X175-16N, symbol formula:74HC4050D,653
- removed U1: MPL3115A2, Package_LGA:NXP_LGA-8_3x5mm_P1.25mm_H1.1mm, symbol Sensor_Pressure:MPL3115A2
- removed U2: LP2985-3.3, Package_TO_SOT_SMD:SOT-23-5, symbol Regulator_Linear:LP2985-3.3
- removed U?: BNO055_BNO055, symbol bno055:BNO055_BNO055
- added C3: 100n, footprints:C_0805_OEM, symbol Device:C
- added TP? (x2): TestPoint, symbol Connector:TestPoint
- added TP? (x2): TestPoint, TestPoint:TestPoint_Keystone_5010-5014_Multipurpose, symbol Connector:TestPoint
- added U1: BNO055, BNO055:BNO055, symbol rev1-rescue:BNO055_BNO055-bno055
- added U?: Teensy3.6, symbol teensy:Teensy3.6
- U2: value ASDMB-xxxMHz -> ASDMB-32kHz
- U?: symbol rocketry:MPL3115A2 -> rev1-rescue:MPL3115A2-rocketry
- gave numbers to parts that had none: 4
- renumbered TP_GND to TP_GND1
Connections:
- net SDL is gone; now on net SDA_TEENSY: U?.7 (SDL)
- net +3V3: now also TP?.1, TP?.1, U1.28 (VDDIO), U1.3 (VDD), U?.51 (3.3V); no longer C1.2, C1.2, C2.1, C2.2, C3.1, C4.2, C5.1, TP_GND1.1, U2.2 (GND), U?.3 (GND)
- net COM3: now also U1.17 (COM3), U?.13 (11_MOSI0)
- net OptionalOSCinput: now also U1.27 (XIN32)
- net OptionalOSCoutput: now also U1.26 (XOUT32)
- net nBOOT_LOAD_PIN: now also U1.4 (nBOOT_LOAD_PIN), U?.4 (2_PWM)
- net nRESET: now also U1.11 (nRESET), U?.8 (6_PWM)
- net at C4.1, TP3.1: now also U1.9 (CAP)
- net at TP1.1, U?.2 (CAP): now also C3.1
- net INT1 renamed INT1_MPL3115A2
- net INT1_MPL3115A2: now also U?.16 (24)
- net INT2 renamed INT2_MPL3115A2
- net INT2_MPL3115A2: now also U?.17 (25)
- net SCL renamed SCL_TEENSY
- net SCL_TEENSY: now also U1.19 (COM1), U?.46 (19_A5_SCL0_TOUCH)
- net SDA renamed SDA_TEENSY
- net SDA_TEENSY: now also U1.20 (COM0), U?.45 (18_A4_SDA0_TOUCH)
- new net GND: C1.2, C1.2, C2.1, C2.2, C3.1, C3.2, C4.2, C5.1, TP?.1, TP?.1, TP_GND1.1, U1.10 (PIN10), U1.16 (PIN16), U1.18 (COM2), U1.2 (GND), U1.25 (GNDIO), U1.5 (PS1), U1.6 (PS0), U1.~ (PIN15), U2.2 (GND), U?.1 (GND), U?.3 (GND)
- new net INT_BNO055: U1.14 (INT), U?.7 (5_PWM_TX1_MISO1)
- no-connect marks 3 -> 0
Other:
- note added: "Altimeter w/ Logic Shifter"
- note added: "BNO055 9-axis w/Logic Shifter\n"
- note added: "notes here\n"
- note added: "put notes here later\n"
- note removed: "Converts Teensy 5V logic signal to 3V for use by altimeter"
- note removed: "I2C Logic Converter"
- moved on the sheet: C1, C2, C3, C4, C5, R1, R2, R3, R4, TP1, TP2, TP3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

Commit message: change BNO055 section of the rev1 schematic to use a two-pin crystal with capacitors
Parts:
- removed C5: 0.01u, footprints:C_0603_1608Metric, symbol Device:C
- removed TP4: TestPoint, symbol Connector:TestPoint
- removed U2: ASDMB-32kHz, ASDK2-32.768KHZ-LR-T3:ASDK2-32.768KHZ-LR-T3, symbol Oscillator:ASDMB-xxxMHz
- added C? (x2): 22pF, Capacitor_SMD:C_0805_2012Metric, symbol Device:C
- added Y?: Crystal_32kHz768, footprints:FC-135_3.2x1.5mm, symbol preferred_parts:Crystal_32kHz768
- U?: symbol teensy:Teensy3.6 -> rev1-rescue:Teensy3.6-teensy
Connections:
- net GND: now also C?.2, C?.2
- net OptionalOSCinput: now also C?.1, Y?.1
- net OptionalOSCoutput: now also C?.1, Y?.2
Other:
- note added: "For the crystal, see BNO055 datasheet page 100."
- note added: "https://cdn-shop.adafruit.com/datasheets/BST_BNO055_DS000_12.pdf"
Changed lines of the file:
@@
-	-1   0    0    1
-$EndComp
-$Comp
-L Connector:TestPoint TP4
-U 1 1 5FEBF50A
-P 10600 2900
-F 0 "TP4" H 10542 2926 50  0000 R CNN
-F 1 "TestPoint" H 10542 3017 50  0000 R CNN
-F 2 "" H 10800 2900 50  0001 C CNN
-F 3 "~" H 10800 2900 50  0001 C CNN
-	1    10600 2900
 	-1   0    0    1
 $EndComp
@@
 $EndComp
 Wire Wire Line
-	10600 2750 10750 2750
-Connection ~ 10600 2750
-Wire Wire Line
-	10600 2900 10600 2750
-Wire Wire Line
-	10450 2750 10600 2750
-Wire Wire Line
 	6650 6950 6450 6950
 Connection ~ 6650 6950
@@
 	-1   0    0    1
 $EndComp
-Connection ~ 9450 2750
-Wire Wire Line
-	9450 3050 9450 2750
-Connection ~ 9900 3050
-Wire Wire Line
-	9750 3050 9900 3050
-$Comp
-L Device:C C5
-U 1 1 5FA6257B
-P 9600 3050
-F 0 "C5" V 9750 3050 50  0000 C CNN
-F 1 "0.01u" V 9450 3050 50  0000 C CNN
-F 2 "footprints:C_0603_1608Metric" H 9638 2900 50  0001 C CNN
-F 3 "~" H 9600 3050 50  0001 C CNN
-	1    9600 3050
-	0    1    1    0
-$EndComp
-Wire Wire Line
-	9900 3050 9900 3200
-Wire Wire Line
-	10150 3050 9900 3050
-$Comp
-L power:GND #PWR03
-U 1 1 5FA5D601
-P 9900 3200
-F 0 "#PWR03" H 9900 2950 50  0001 C CNN
-F 1 "GND" H 9905 3027 50  0000 C CNN
-F 2 "" H 9900 3200 50  0001 C CNN
-F 3 "" H 9900 3200 50  0001 C CNN
-	1    9900 3200
-	1    0    0    -1
-$EndComp
-Wire Wire Line
-	9850 2300 9450 2300
-Connection ~ 9850 2300
-Wire Wire Line
-	9850 2200 9850 2300
-$Comp
-L power:+3.3V #PWR02
-U 1 1 5FA5A832
-P 9850 2200
-F 0 "#PWR02" H 9850 2050 50  0001 C CNN
-F 1 "+3.3V" H 9865 2373 50  0000 C CNN
-F 2 "" H 9850 2200 50  0001 C CNN
-F 3 "" H 9850 2200 50  0001 C CNN
-	1    9850 2200
-	1    0    0    -1
-$EndComp
 $Comp
 L power:+3.3V #PWR01
@@
 F 3 "" H 2050 2350 50  0001 C CNN
 	1    2050 2350
-	1    0    0    -1
-$EndComp
-Wire Wire Line
-	9450 2750 9650 2750
-Wire Wire Line
-	9450 2300 9450 2750
-Wire Wire Line
-	10150 2300 9850 2300
-Wire Wire Line
-	10150 2450 10150 2300
-Text GLabel 10750 2750 2    50   Input ~ 0
-OptionalOSCinput
-$Comp
-L Oscillator:ASDMB-xxxMHz U2
-U 1 1 5FA4E8B7
-P 10050 2750
-F 0 "U2" H 10450 3050 50  0000 L CNN
-F 1 "ASDMB-32kHz" H 10400 3150 50  0000 L CNN
-F 2 "ASDK2-32.768KHZ-LR-T3:ASDK2-32.768KHZ-LR-T3" H 10050 2750 50  0001 C CNN
-F 3 "https://abracon.com/Oscillators/ASDK.pdf" H 10350 3200 50  0001 C CNN
-	1    10050 2750
 	1    0    0    -1
 $EndComp
@@
 Vdd: power supply connection (1.95-3.6V)\nCAP: Ext. capacitor\nGND: Ground\nVddio: Digital interface power supply (1.62-3.6V)\nINT2: Pressure interrupt 2\nINT1: Pressure interrupt 1\nSDA: I2C serial data\nSDL: I2C serial clock
 $Comp
-L teensy:Teensy3.6 U?
+L rev1-rescue:Teensy3.6-teensy U?
 U 1 1 60876FE4
 P 28550 4950
@@
 Text GLabel 4400 8250 1    39   Input ~ 0
 VIN_TEENSY
+$Comp
+L preferred_parts:Crystal_32kHz768 Y?
+U 1 1 6002B9D1
+P 10900 2100
+F 0 "Y?" V 10854 2231 50  0000 L CNN
+F 1 "Crystal_32kHz768" V 10945 2231 50  0000 L CNN
+F 2 "footprints:FC-135_3.2x1.5mm" H 10850 2175 50  0001 C CNN
+F 3 "https://support.epson.biz/td/api/doc_check.php?dl=brief_FC-135&lang=en" H 10950 2275 50  0001 C CNN
+F 4 "DK" H 10850 2300 60  0001 C CNN "MFN"
+F 5 "SER4084CT-ND" H 10900 2350 60  0001 C CNN "MPN"
+F 6 "https://www.digikey.com/product-detail/en/epson/FC-135-32.7680KA-AC0/SER4084CT-ND/6132704" H 11350 2675 60  0001 C CNN "PurchasingLink"
+	1    10900 2100
+	0    1    1    0
+$EndComp
+$Comp
+L Device:C C?
+U 1 1 6002E87E
+P 10350 1800
+F 0 "C?" V 10098 1800 50  0000 C CNN
+F 1 "22pF" V 10189 1800 50  0000 C CNN
+F 2 "Capacitor_SMD:C_0805_2012Metric" H 10388 1650 50  0001 C CNN
+F 3 "~" H 10350 1800 50  0001 C CNN
+	1    10350 1800
+	0    1    1    0
+$EndComp
+$Comp
+L Device:C C?
+U 1 1 600377E0
+P 10350 2500
+F 0 "C?" V 10098 2500 50  0000 C CNN
+F 1 "22pF" V 10189 2500 50  0000 C CNN
+F 2 "Capacitor_SMD:C_0805_2012Metric" H 10388 2350 50  0001 C CNN
+F 3 "~" H 10350 2500 50  0001 C CNN
+	1    10350 2500
+	0    1    1    0
+$EndComp
+Wire Wire Line
+	10900 1950 10900 1800
+Wire Wire Line
+	10900 1800 10500 1800
+Wire Wire Line
+	10900 2250 10900 2500
+Wire Wire Line
+	10900 2500 10500 2500
+Text GLabel 11800 1800 2    50   Input ~ 0
+OptionalOSCinput
+Text GLabel 11800 2500 2    50   Input ~ 0
+OptionalOSCoutput
+Wire Wire Line
+	11800 1800 10900 1800
+Connection ~ 10900 1800
+Wire Wire Line
+	11800 2500 10900 2500
+Connection ~ 10900 2500
+$Comp
+L power:GND #PWR?
+U 1 1 60053EEF
+P 9850 2850
+F 0 "#PWR?" H 9850 2600 50  0001 C CNN
+F 1 "GND" H 9855 2677 50  0000 C CNN
+F 2 "" H 9850 2850 50  0001 C CNN
+F 3 "" H 9850 2850 50  0001 C CNN
+	1    9850 2850
+	1    0    0    -1
+$EndComp
+Wire Wire Line
+	10200 2500 9850 2500
+Wire Wire Line
+	9850 2500 9850 2850
+Wire Wire Line
+	10200 1800 9850 1800
+Wire Wire Line
+	9850 1800 9850 2500
+Connection ~ 9850 2500
+Text Notes 11000 1400 0    50   ~ 0
+For the crystal, see BNO055 datasheet page 100.
+Text Notes 10700 1550 0    50   ~ 0
+https://cdn-shop.adafruit.com/datasheets/BST_BNO055_DS000_12.pdf
 $EndSCHEMATC

Commit message: fix annotation
Parts:
- C5, C6: renamed from C?; value 22pF -> 22p
- gave numbers to parts that had none: 7
- renumbered C1 to C7, C2 to C8, C3 to C9, TP1 to TP8
Changed lines of the file:
@@
 $EndDescr
 $Comp
-L rev1-rescue:MPL3115A2-rocketry U?
+L rev1-rescue:MPL3115A2-rocketry U2
 U 1 1 5FF5B454
 P 18350 2950
-F 0 "U?" H 18350 3615 50  0000 C CNN
+F 0 "U2" H 18350 3615 50  0000 C CNN
 F 1 "MPL3115A2" H 18350 3524 50  0000 C CNN
 F 2 "" H 18350 2950 50  0001 C CNN
@@
 $EndComp
 $Comp
-L Device:C C2
+L Device:C C8
 U 1 1 60279C52
 P 17100 2650
-F 0 "C2" H 17215 2696 50  0000 L CNN
+F 0 "C8" H 17215 2696 50  0000 L CNN
 F 1 "10u" H 17215 2605 50  0000 L CNN
 F 2 "footprints:C_0805_OEM" H 17138 2500 50  0001 C CNN
@@
 $EndComp
 $Comp
-L Device:C C1
+L Device:C C7
 U 1 1 5F97B20B
 P 16600 2650
-F 0 "C1" H 16715 2696 50  0000 L CNN
+F 0 "C7" H 16715 2696 50  0000 L CNN
 F 1 "100n" H 16715 2605 50  0000 L CNN
 F 2 "footprints:C_0805_OEM" H 16638 2500 50  0001 C CNN
@@
 Connection ~ 17100 3050
 $Comp
-L Device:C C3
+L Device:C C9
 U 1 1 60279C54
 P 17500 2900
-F 0 "C3" H 17615 2946 50  0000 L CNN
+F 0 "C9" H 17615 2946 50  0000 L CNN
 F 1 "100n" H 17615 2855 50  0000 L CNN
 F 2 "footprints:C_0805_OEM" H 17538 2750 50  0001 C CNN
@@
 	19750 2850 19750 2750
 $Comp
-L Connector:TestPoint TP1
+L Connector:TestPoint TP8
 U 1 1 5FEA9553
 P 17600 1850
-F 0 "TP1" H 17658 1968 50  0000 L CNN
+F 0 "TP8" H 17658 1968 50  0000 L CNN
 F 1 "TestPoint" H 17658 1877 50  0000 L CNN
 F 2 "TestPoint:TestPoint_Keystone_5010-5014_Multipurpose" H 17800 1850 50  0001 C CNN
@@
 Connection ~ 20150 2850
 $Comp
-L Connector:TestPoint TP?
+L Connector:TestPoint TP6
 U 1 1 60279C64
 P 20950 2850
-F 0 "TP?" H 21008 2968 50  0000 L CNN
+F 0 "TP6" H 21008 2968 50  0000 L CNN
 F 1 "TestPoint" H 21008 2877 50  0000 L CNN
 F 2 "TestPoint:TestPoint_Keystone_5010-5014_Multipurpose" H 21150 2850 50  0001 C CNN
@@
 $EndComp
 $Comp
-L Connector:TestPoint TP?
+L Connector:TestPoint TP7
 U 1 1 60279C65
 P 20950 3000
-F 0 "TP?" H 21008 3118 50  0000 L CNN
+F 0 "TP7" H 21008 3118 50  0000 L CNN
 F 1 "TestPoint" H 21008 3027 50  0000 L CNN
 F 2 "TestPoint:TestPoint_Keystone_5010-5014_Multipurpose" H 21150 3000 50  0001 C CNN
@@
 	20550 3000 20950 3000
 $Comp
-L power:PWR_FLAG #FLG?
+L power:PWR_FLAG #FLG0106
 U 1 1 60279C66
 P 19750 3100
-F 0 "#FLG?" H 19750 3175 50  0001 C CNN
+F 0 "#FLG0106" H 19750 3175 50  0001 C CNN
 F 1 "PWR_FLAG" H 19750 3273 50  0000 C CNN
 F 2 "" H 19750 3100 50  0001 C CNN
@@
 $EndComp
 $Comp
-L power:+3.3V #PWR0104
+L power:+3.3V #PWR0107
 U 1 1 5FED1CED
 P 2950 8250
-F 0 "#PWR0104" H 2950 8100 50  0001 C CNN
+F 0 "#PWR0107" H 2950 8100 50  0001 C CNN
 F 1 "+3.3V" H 2965 8423 50  0000 C CNN
 F 2 "" H 2950 8250 50  0001 C CNN
@@
 $EndComp
 $Comp
-L power:GNDPWR #PWR0103
+L power:GNDPWR #PWR0108
 U 1 1 5FEC5490
 P 1400 8550
-F 0 "#PWR0103" H 1400 8350 50  0001 C CNN
+F 0 "#PWR0108" H 1400 8350 50  0001 C CNN
 F 1 "GNDPWR" H 1404 8396 50  0000 C CNN
 F 2 "" H 1400 8500 50  0001 C CNN
@@
 Connection ~ 2050 2750
 $Comp
-L power:PWR_FLAG #FLG0101
+L power:PWR_FLAG #FLG0107
 U 1 1 5F8BC0A5
 P 2050 2750
-F 0 "#FLG0101" H 2050 2825 50  0001 C CNN
+F 0 "#FLG0107" H 2050 2825 50  0001 C CNN
 F 1 "PWR_FLAG" V 2050 2877 50  0000 L CNN
 F 2 "" H 2050 2750 50  0001 C CNN
@@
 	0    -1   -1   0
 $EndComp
-Text GLabel 950  8250 1    50   Input ~ 0
-GND
 Wire Wire Line
 	2050 2450 2050 2350
@@
 	7150 6950 6650 6950
 $Comp
-L power:GND #PWR0101
+L power:GND #PWR0109
 U 1 1 5F894FED
 P 6450 6950
-F 0 "#PWR0101" H 6450 6700 50  0001 C CNN
+F 0 "#PWR0109" H 6450 6700 50  0001 C CNN
 F 1 "GND" H 6455 6777 50  0000 C CNN
 F 2 "" H 6450 6950 50  0001 C CNN
@@
 $EndComp
 $Comp
-L Connector:TestPoint TP?
+L Connector:TestPoint TP5
 U 1 1 5FF680D8
 P 3850 8550
-F 0 "TP?" H 3792 8576 50  0000 R CNN
+F 0 "TP5" H 3792 8576 50  0000 R CNN
 F 1 "TestPoint" H 3792 8667 50  0000 R CNN
 F 2 "" H 4050 8550 50  0001 C CNN
@@
 $EndComp
 $Comp
-L Connector:TestPoint TP?
+L Connector:TestPoint TP4
 U 1 1 5FF68D98
 P 1850 8250
-F 0 "TP?" H 1792 8276 50  0000 R CNN
+F 0 "TP4" H 1792 8276 50  0000 R CNN
 F 1 "TestPoint" H 1792 8367 50  0000 R CNN
 F 2 "" H 2050 8250 50  0001 C CNN
@@
 	3850 8550 3850 8400
 Connection ~ 3850 8400
-Wire Wire Line
-	950  8250 950  8450
-Connection ~ 950  8450
 Wire Wire Line
 	9250 5950 9250 6950
@@
 Vdd: power supply connection (1.95-3.6V)\nCAP: Ext. capacitor\nGND: Ground\nVddio: Digital interface power supply (1.62-3.6V)\nINT2: Pressure interrupt 2\nINT1: Pressure interrupt 1\nSDA: I2C serial data\nSDL: I2C serial clock
 $Comp
-L rev1-rescue:Teensy3.6-teensy U?
+L rev1-rescue:Teensy3.6-teensy U3
 U 1 1 60876FE4
 P 28550 4950
-F 0 "U?" H 28550 7387 60  0000 C CNN
+F 0 "U3" H 28550 7387 60  0000 C CNN
 F 1 "Teensy3.6" H 28550 7281 60  0000 C CNN
 F 2 "" H 28550 5000 60  0000 C CNN
@@
 VIN_TEENSY
 $Comp
-L power:+3.3V #PWR0102
+L power:+3.3V #PWR0110
 U 1 1 5FA181ED
 P 16600 2350
-F 0 "#PWR0102" H 16600 2200 50  0001 C CNN
+F 0 "#PWR0110" H 16600 2200 50  0001 C CNN
 F 1 "+3.3V" H 16615 2523 50  0000 C CNN
 F 2 "" H 16600 2350 50  0001 C CNN
@@
 VIN_TEENSY
 $Comp
-L preferred_parts:Crystal_32kHz768 Y?
+L preferred_parts:Crystal_32kHz768 Y1
 U 1 1 6002B9D1
 P 10900 2100
-F 0 "Y?" V 10854 2231 50  0000 L CNN
+F 0 "Y1" V 10854 2231 50  0000 L CNN
 F 1 "Crystal_32kHz768" V 10945 2231 50  0000 L CNN
 F 2 "footprints:FC-135_3.2x1.5mm" H 10850 2175 50  0001 C CNN
@@
 $EndComp
 $Comp
-L Device:C C?
+L Device:C C5
 U 1 1 6002E87E
 P 10350 1800
-F 0 "C?" V 10098 1800 50  0000 C CNN
-F 1 "22pF" V 10189 1800 50  0000 C CNN
+F 0 "C5" V 10098 1800 50  0000 C CNN
+F 1 "22p" V 10189 1800 50  0000 C CNN
 F 2 "Capacitor_SMD:C_0805_2012Metric" H 10388 1650 50  0001 C CNN
 F 3 "~" H 10350 1800 50  0001 C CNN
@@
 $EndComp
 $Comp
-L Device:C C?
+L Device:C C6
 U 1 1 600377E0
 P 10350 2500
-F 0 "C?" V 10098 2500 50  0000 C CNN
-F 1 "22pF" V 10189 2500 50  0000 C CNN
+F 0 "C6" V 10098 2500 50  0000 C CNN
+F 1 "22p" V 10189 2500 50  0000 C CNN
 F 2 "Capacitor_SMD:C_0805_2012Metric" H 10388 2350 50  0001 C CNN
 F 3 "~" H 10350 2500 50  0001 C CNN
@@
 Connection ~ 10900 2500
 $Comp
-L power:GND #PWR?
+L power:GND #PWR0111
 U 1 1 60053EEF
 P 9850 2850
-F 0 "#PWR?" H 9850 2600 50  0001 C CNN
+F 0 "#PWR0111" H 9850 2600 50  0001 C CNN
 F 1 "GND" H 9855 2677 50  0000 C CNN
 F 2 "" H 9850 2850 50  0001 C CNN

Commit message: add abd change footprints
Parts:
- C5, C6: footprint Capacitor_SMD:C_0805_2012Metric -> footprints:C_0805_OEM
- TP1, TP2, TP3, TP4, TP5, TP_GND1: footprint (none) -> footprints:Test_Point_D1.02mm
- TP6, TP7, TP8: footprint TestPoint:TestPoint_Keystone_5010-5014_Multipurpose -> footprints:Test_Point_D1.02mm
- U2: footprint (none) -> MPL3115A2_barometer:MPL3115A2
- U3: footprint (none) -> footprints:Teensy3-6
Changed lines of the file:
@@
 F 0 "U2" H 18350 3615 50  0000 C CNN
 F 1 "MPL3115A2" H 18350 3524 50  0000 C CNN
-F 2 "" H 18350 2950 50  0001 C CNN
+F 2 "MPL3115A2_barometer:MPL3115A2" H 18350 2950 50  0001 C CNN
 F 3 "" H 18350 2950 50  0001 C CNN
 	1    18350 2950
@@
 F 0 "TP8" H 17658 1968 50  0000 L CNN
 F 1 "TestPoint" H 17658 1877 50  0000 L CNN
-F 2 "TestPoint:TestPoint_Keystone_5010-5014_Multipurpose" H 17800 1850 50  0001 C CNN
+F 2 "footprints:Test_Point_D1.02mm" H 17800 1850 50  0001 C CNN
 F 3 "~" H 17800 1850 50  0001 C CNN
 	1    17600 1850
@@
 F 0 "TP6" H 21008 2968 50  0000 L CNN
 F 1 "TestPoint" H 21008 2877 50  0000 L CNN
-F 2 "TestPoint:TestPoint_Keystone_5010-5014_Multipurpose" H 21150 2850 50  0001 C CNN
+F 2 "footprints:Test_Point_D1.02mm" H 21150 2850 50  0001 C CNN
 F 3 "~" H 21150 2850 50  0001 C CNN
 	1    20950 2850
@@
 F 0 "TP7" H 21008 3118 50  0000 L CNN
 F 1 "TestPoint" H 21008 3027 50  0000 L CNN
-F 2 "TestPoint:TestPoint_Keystone_5010-5014_Multipurpose" H 21150 3000 50  0001 C CNN
+F 2 "footprints:Test_Point_D1.02mm" H 21150 3000 50  0001 C CNN
 F 3 "~" H 21150 3000 50  0001 C CNN
 	1    20950 3000
@@
 F 0 "TP2" H 2792 5226 50  0000 R CNN
 F 1 "TestPoint" H 2792 5317 50  0000 R CNN
-F 2 "" H 3050 5200 50  0001 C CNN
+F 2 "footprints:Test_Point_D1.02mm" H 3050 5200 50  0001 C CNN
 F 3 "~" H 3050 5200 50  0001 C CNN
 	1    2850 5200
@@
 F 0 "TP3" H 5242 7926 50  0000 R CNN
 F 1 "TestPoint" H 5242 8017 50  0000 R CNN
-F 2 "" H 5500 7900 50  0001 C CNN
+F 2 "footprints:Test_Point_D1.02mm" H 5500 7900 50  0001 C CNN
 F 3 "~" H 5500 7900 50  0001 C CNN
 	1    5300 7900
@@
 F 0 "TP1" H 2642 7576 50  0000 R CNN
 F 1 "TestPoint" H 2642 7667 50  0000 R CNN
-F 2 "" H 2900 7550 50  0001 C CNN
+F 2 "footprints:Test_Point_D1.02mm" H 2900 7550 50  0001 C CNN
 F 3 "~" H 2900 7550 50  0001 C CNN
 	1    2700 7550
@@
 F 0 "TP_GND1" H 6592 6976 50  0000 R CNN
 F 1 "TestPoint" H 6592 7067 50  0000 R CNN
-F 2 "" H 6850 6950 50  0001 C CNN
+F 2 "footprints:Test_Point_D1.02mm" H 6850 6950 50  0001 C CNN
 F 3 "~" H 6850 6950 50  0001 C CNN
 	1    6650 6950
@@
 F 0 "TP5" H 3792 8576 50  0000 R CNN
 F 1 "TestPoint" H 3792 8667 50  0000 R CNN
-F 2 "" H 4050 8550 50  0001 C CNN
+F 2 "footprints:Test_Point_D1.02mm" H 4050 8550 50  0001 C CNN
 F 3 "~" H 4050 8550 50  0001 C CNN
 	1    3850 8550
@@
 F 0 "TP4" H 1792 8276 50  0000 R CNN
 F 1 "TestPoint" H 1792 8367 50  0000 R CNN
-F 2 "" H 2050 8250 50  0001 C CNN
+F 2 "footprints:Test_Point_D1.02mm" H 2050 8250 50  0001 C CNN
 F 3 "~" H 2050 8250 50  0001 C CNN
 	1    1850 8250
@@
 F 0 "U3" H 28550 7387 60  0000 C CNN
 F 1 "Teensy3.6" H 28550 7281 60  0000 C CNN
-F 2 "" H 28550 5000 60  0000 C CNN
+F 2 "footprints:Teensy3-6" H 28550 5000 60  0001 C CNN
 F 3 "" H 28550 5000 60  0000 C CNN
 	1    28550 4950
@@
 F 0 "C5" V 10098 1800 50  0000 C CNN
 F 1 "22p" V 10189 1800 50  0000 C CNN
-F 2 "Capacitor_SMD:C_0805_2012Metric" H 10388 1650 50  0001 C CNN
+F 2 "footprints:C_0805_OEM" H 10388 1650 50  0001 C CNN
 F 3 "~" H 10350 1800 50  0001 C CNN
 	1    10350 1800
@@
 F 0 "C6" V 10098 2500 50  0000 C CNN
 F 1 "22p" V 10189 2500 50  0000 C CNN
-F 2 "Capacitor_SMD:C_0805_2012Metric" H 10388 2350 50  0001 C CNN
+F 2 "footprints:C_0805_OEM" H 10388 2350 50  0001 C CNN
 F 3 "~" H 10350 2500 50  0001 C CNN
 	1    10350 2500

Commit message: wip
Parts:
- added TP10, TP9: TestPoint, footprints:Test_Point_D1.02mm, symbol Connector:TestPoint
Connections:
- net OptionalOSCinput: now also TP9.1
- net OptionalOSCoutput: now also TP10.1
Changed lines of the file:
@@
 OptionalOSCoutput
 Wire Wire Line
-	11800 1800 10900 1800
+	11800 1800 11400 1800
 Connection ~ 10900 1800
 Wire Wire Line
-	11800 2500 10900 2500
+	11800 2500 11400 2500
 Connection ~ 10900 2500
 $Comp
@@
 Text Notes 10700 1550 0    50   ~ 0
 https://cdn-shop.adafruit.com/datasheets/BST_BNO055_DS000_12.pdf
+$Comp
+L Connector:TestPoint TP10
+U 1 1 600A3D96
+P 11400 2500
+F 0 "TP10" H 11342 2526 50  0000 R CNN
+F 1 "TestPoint" H 11342 2617 50  0000 R CNN
+F 2 "footprints:Test_Point_D1.02mm" H 11600 2500 50  0001 C CNN
+F 3 "~" H 11600 2500 50  0001 C CNN
+	1    11400 2500
+	-1   0    0    1
+$EndComp
+Connection ~ 11400 2500
+Wire Wire Line
+	11400 2500 10900 2500
+$Comp
+L Connector:TestPoint TP9
+U 1 1 600A5053
+P 11400 1800
+F 0 "TP9" H 11342 1826 50  0000 R CNN
+F 1 "TestPoint" H 11342 1917 50  0000 R CNN
+F 2 "footprints:Test_Point_D1.02mm" H 11600 1800 50  0001 C CNN
+F 3 "~" H 11600 1800 50  0001 C CNN
+	1    11400 1800
+	1    0    0    -1
+$EndComp
+Connection ~ 11400 1800
+Wire Wire Line
+	11400 1800 10900 1800
 $EndSCHEMATC

Commit message: wip
Connections:
- net SCL_TEENSY: now also U3.9 (7_RX3_MISO0_SCL0)
- net SDA_TEENSY: now also U3.10 (8_TX3_MISO0_SDA0)
Changed lines of the file:
@@
 Wire Wire Line
 	11400 1800 10900 1800
+Text GLabel 27400 3600 0    39   Input ~ 0
+SCL_TEENSY
+Text GLabel 27400 3700 0    39   Input ~ 0
+SDA_TEENSY
 $EndSCHEMATC

Commit message: wip
Connections:
- net +3V3: now also U3.15 (3.3V); no longer U3.51 (3.3V)
- net INT1_MPL3115A2: now also U3.17 (25); no longer U3.16 (24)
- net INT2_MPL3115A2: now also U3.16 (24); no longer U3.17 (25)
- net SCL_TEENSY: no longer U3.46 (19_A5_SCL0_TOUCH)
- net SDA_TEENSY: no longer U3.45 (18_A4_SDA0_TOUCH)
Changed lines of the file:
@@
 Text Label 27400 2800 2    118  ~ 0
 GND
-Text GLabel 29700 6500 2    39   Input ~ 0
+Text GLabel 27400 4200 0    39   Input ~ 0
 VIN_TEENSY
-Text GLabel 29700 7100 2    39   Input ~ 0
-SDA_TEENSY
-Text GLabel 29700 7000 2    39   Input ~ 0
-SCL_TEENSY
 Wire Wire Line
 	6900 7300 9850 7300
 Text GLabel 9850 7300 2    50   Input ~ 0
 INT_BNO055
+Text GLabel 27400 4400 0    50   Input ~ 0
+INT1_MPL3115A2
 Text GLabel 27400 4300 0    50   Input ~ 0
-INT1_MPL3115A2
-Text GLabel 27400 4400 0    50   Input ~ 0
 INT2_MPL3115A2
 Text GLabel 27400 3500 0    50   Input ~ 0
