File: hardware/BNO055/BNO055_circuit_i2C.sch (KiCad schematic (older format))
At the start: 18 parts, among them U1 BNO055, U2 ASDMB-xxxMHz

Commit message: add level shifter to BNO055 schematic. Needs review
Parts:
- added TP? (x2): TestPoint, symbol Connector:TestPoint
- added U? (x2): 74HC4050D,653, SOIC127P600X175-16N, symbol preferred_parts:74HC4050D,653
- H1, H2: symbol BNO055_circuit_i2C-rescue:Header_2x3-Olin_Rocketry_Symbols -> preferred_parts:CONN_02X03
- U2: value ASDMB-xxxMHz -> ASDMB-32kHz
- gave numbers to parts that had none: 4
- renumbered TP_GND to TP_GND1
Connections:
- net labels added: COM3_TO_MC, INT_TO_MC, SCL_TO_MC, SDA_TO_MC, VCC, nBOOT_LOAD_TO_MC, nRESET_TO_MC
- wire segments 113 -> 122
- no-connect marks 1 -> 0
Other:
- note added: "Stepping down potentially 5V Vcc to 3V Vdd and Vddio"

Commit message: add level shifter to MLP3115A2. Needs review
Parts:
- H1, H2: symbol preferred_parts:CONN_02X03 -> BNO055_circuit_i2C-rescue:CONN_02X03-preferred_parts
- U? (x2): symbol preferred_parts:74HC4050D,653 -> BNO055_circuit_i2C-rescue:74HC4050D,653-preferred_parts
Changed lines of the file:
@@
 $EndDescr
 $Comp
-L preferred_parts:74HC4050D,653 U?
+L BNO055_circuit_i2C-rescue:74HC4050D,653-preferred_parts U?
 U 1 1 5FF3A250
 P 12750 5900
@@
 $EndComp
 $Comp
-L preferred_parts:CONN_02X03 H2
+L BNO055_circuit_i2C-rescue:CONN_02X03-preferred_parts H2
 U 1 1 5F967DE8
 P 10100 5300
@@
 $EndComp
 $Comp
-L preferred_parts:CONN_02X03 H1
+L BNO055_circuit_i2C-rescue:CONN_02X03-preferred_parts H1
 U 1 1 5F967336
 P 10050 4600
@@
 $EndComp
 $Comp
-L preferred_parts:74HC4050D,653 U?
+L BNO055_circuit_i2C-rescue:74HC4050D,653-preferred_parts U?
 U 1 1 5FF66BE6
 P 12750 3750
