File: hardware/rev2/rev2.sch (KiCad schematic (older format))
At the start: 43 parts, among them J1 Conn_01x09_Female, J2 RFM9X_header, J3 Conn_01x03_Male, Q1 Q_PNP_BCE, U1 BNO055, U2 MPL3115A2, U3 Teensy3.6, U4 BMI088, U5 ADXL345BCCZ, Y1 Crystal_32kHz768

Commit message: copy Rev1 into Rev2. Change power input circuit from using MOSFET to TPS2113
Parts:
- removed D2, D3: D, footprints:D_0805_OEM, symbol Device:D
- removed Q1: Q_PNP_BCE, Package_TO_SOT_THT:TO-220-3_Horizontal_TabDown, symbol Device:Q_PNP_BCE
- removed R5: 1K, footprints:R_0805_OEM, symbol preferred_parts:R_1.07K
- added C14: C_1uF, footprints:C_0805_OEM, symbol preferred_parts:C_1uF
- added R5: R_20k, footprints:R_0805_OEM, symbol preferred_parts:R_475
- added R6: R_8k, footprints:R_0805_OEM, symbol preferred_parts:R_475
- added R7: R_475, footprints:R_0805_OEM, symbol preferred_parts:R_475
- added U6: BNO055, Package_LGA:LGA-28_5.2x3.8mm_P0.5mm, symbol Sensor_Motion:BNO055
- added U7: TPS2113ADRBR, footprints:TPS2113ADRBR, symbol preferred_parts:TPS2113ADRBR
- added U8: MPL3115A2, Package_LGA:NXP_LGA-8_3x5mm_P1.25mm_H1.1mm, symbol Sensor_Pressure:MPL3115A2
- U1: symbol rev1-rescue:BNO055_BNO055-bno055 -> BNO055:BNO055
- U2: symbol rev1-rescue:MPL3115A2-rocketry -> MPL3115A2:MPL3115A2
- U3: symbol rev1-rescue:Teensy3.6-teensy -> rev2-rescue:Teensy3.6-teensy-rev1-rescue
Connections:
- wire segments 204 -> 216
- no-connect marks 68 -> 69
Other:
- note added: "Ratio of R5 to R6 has to be 2.5 to 1\n(or rather 2.0 to 0.8) \nso that VSNS receives 0.8V when\nBMS_to_sensors drops below 2.8V"
- note removed: "notes here\n"
- note removed: "put notes here later\n"
- moved on the sheet: BMS_CONN1, BMS_CONN2, D1, J3

Commit message: Remove BNO055 and BMI055 from Rev2 schematic. Add 4.99K pull up resistors for SCL and SDA lines
Parts:
- removed BOOT1, CAP1, OSCin1, OSCout1, nReset1: TestPoint, footprints:Test-Point-Pin_Drill2.79mm, symbol Connector:TestPoint
- removed C1, C4: 100n, footprints:C_0805_OEM, symbol Device:C
- removed C12, C13: 100n, footprints:C_0805_OEM, symbol preferred_parts:C_100nF
- removed C2: 6.8n, footprints:C_0805_OEM, symbol Device:C
- removed C3: 120n, footprints:C_0805_OEM, symbol Device:C
- removed C5, C6: 22p, footprints:C_0805_OEM, symbol Device:C
- removed R1, R2, R3, R4: 10k, footprints:R_0805_OEM, symbol Device:R
- removed U1: BNO055, BNO055:BNO055, symbol BNO055:BNO055
- removed U4: BMI088, footprints:bmi088, symbol preferred_parts:BMI088
- removed U6: BNO055, Package_LGA:LGA-28_5.2x3.8mm_P0.5mm, symbol Sensor_Motion:BNO055
- removed U8: MPL3115A2, Package_LGA:NXP_LGA-8_3x5mm_P1.25mm_H1.1mm, symbol Sensor_Pressure:MPL3115A2
- removed Y1: Crystal_32kHz768, footprints:FC-135_3.2x1.5mm, symbol preferred_parts:Crystal_32kHz768
- added R? (x2): R_4.99K, footprints:R_0805_OEM, symbol preferred_parts:R_4.99K
- J2: symbol preferred_parts:RFM9X_header -> rev2-rescue:RFM9X_header-preferred_parts
Connections:
- net labels removed: GNDIO, INTERRUPT, OptionalOSCinput, OptionalOSCoutput, SCL, SDA, VDD, VDDIO
- wire segments 216 -> 113
- no-connect marks 69 -> 68
Other:
- note removed: "BMI088"
- note removed: "BNO055 9-axis Accelerometer\n"
- note removed: "For the crystal, see BNO055 datasheet page 100."
- note removed: "These pull-up resistors (R3 and R4) should arguably be\nin a separate location on the schematic, as they affect\nthe entire I2C bus, not just the BNO055"
- note removed: "VDDIO"
- note removed: "https://cdn-shop.adafruit.com/datasheets/BST_BNO055_DS000_12.pdf"
- moved on the sheet: C7, C8, C9, CAP2, GND1, GND2, U2, VDD1, VDD2

Commit message: fix some DRC errors
Parts:
- gave numbers to parts that had none: 2
Connections:
- net 3.3VBMS is gone; now on net +3V3: C14.1, U7.7 (OUT)
- net SCL_TEENSY: now also U3.46 (19_A5_SCL0_TOUCH)
- net SDA_TEENSY: now also U3.45 (18_A4_SDA0_TOUCH)
- net A0_ACCEL_BMI088: no longer names the net of U3.19 (27_RX1)
- net A0_GYRO_BMI088: no longer names the net of U3.18 (26_TX1)
- net COM3: no longer names the net of U3.9 (7_RX3_MISO0_SCL0)
- net INT1_ACCEL_BMI088: no longer names the net of U3.24 (32_A13_TX4_SCK1)
- net INT2_ACCEL_BMI088: no longer names the net of U3.21 (29_PWM_CAN0TX_TOUCH)
- net INT3_GYRO_BMI088: no longer names the net of U3.22 (30_PWM_CAN0RX_TOUCH)
- net INT4_GYRO_BMI088: no longer names the net of U3.23 (31_A12_RX4_CS1)
- net INT_BNO055: no longer names the net of U3.10 (8_TX3_MISO0_SDA0)
- net nBOOT_LOAD_PIN: no longer names the net of U3.12 (10_PWM_TX2_CS0)
- net nRESET: no longer names the net of U3.11 (9_PWM_RX2_CS0)
- no-connect marks 68 -> 76
Changed lines of the file:
@@
 Text GLabel 27650 7200 0    50   Input ~ 0
 INT2_MPL3115A2
-Text GLabel 27650 7500 0    50   Input ~ 0
-nRESET
-Text GLabel 27650 7400 0    50   Input ~ 0
-INT_BNO055
-Text GLabel 27650 7600 0    50   Input ~ 0
-nBOOT_LOAD_PIN
-Text GLabel 27650 7300 0    50   Input ~ 0
-COM3
 $Comp
 L power:+3.3V #PWR0110
@@
 NoConn ~ 27650 10700
 NoConn ~ 27650 10800
-NoConn ~ 29950 10800
-NoConn ~ 29950 10700
 NoConn ~ 29950 10600
 NoConn ~ 29950 10500
@@
 Text GLabel 27650 6700 0    50   Input ~ 0
 INT2_ADXL345
-Text GLabel 27650 8800 0    50   Input ~ 0
-INT1_ACCEL_BMI088
-Text GLabel 27650 8500 0    50   Input ~ 0
-INT2_ACCEL_BMI088
-Text GLabel 27650 8600 0    50   Input ~ 0
-INT3_GYRO_BMI088
-Text GLabel 27650 8700 0    50   Input ~ 0
-INT4_GYRO_BMI088
-Text GLabel 27650 8200 0    50   Input ~ 0
-A0_GYRO_BMI088
-Text GLabel 27650 8300 0    50   Input ~ 0
-A0_ACCEL_BMI088
 Text GLabel 27650 9400 0    50   Input ~ 0
 RX
@@
 	1850 19400 1850 19150
 Wire Wire Line
-	1850 19150 2050 19150
+	1850 19150 2000 19150
 Wire Wire Line
 	1750 19400 1750 18900
@@
 Connection ~ 14100 20750
 $Comp
-L preferred_parts:R_4.99K R?
+L preferred_parts:R_4.99K R1
 U 1 1 6063CB2A
 P 17900 18850
-F 0 "R?" H 17970 18896 50  0000 L CNN
+F 0 "R1" H 17970 18896 50  0000 L CNN
 F 1 "R_4.99K" H 17970 18805 50  0000 L CNN
 F 2 "footprints:R_0805_OEM" H 17700 18800 50  0001 C CNN
@@
 $EndComp
 $Comp
-L preferred_parts:R_4.99K R?
+L preferred_parts:R_4.99K R2
 U 1 1 6063DCFA
 P 19000 18850
-F 0 "R?" H 19070 18896 50  0000 L CNN
+F 0 "R2" H 19070 18896 50  0000 L CNN
 F 1 "R_4.99K" H 19070 18805 50  0000 L CNN
 F 2 "footprints:R_0805_OEM" H 18800 18800 50  0001 C CNN
@@
 $EndComp
 $Comp
-L bno055:+3.3V #PWR?
+L bno055:+3.3V #PWR01
 U 1 1 6063E692
 P 17900 18350
-F 0 "#PWR?" H 17900 18200 50  0001 C CNN
+F 0 "#PWR01" H 17900 18200 50  0001 C CNN
 F 1 "+3.3V" H 17915 18523 50  0000 C CNN
 F 2 "" H 17900 18350 50  0001 C CNN
@@
 $EndComp
 $Comp
-L bno055:+3.3V #PWR?
+L bno055:+3.3V #PWR03
 U 1 1 6063F891
 P 19000 18350
-F 0 "#PWR?" H 19000 18200 50  0001 C CNN
+F 0 "#PWR03" H 19000 18200 50  0001 C CNN
 F 1 "+3.3V" H 19015 18523 50  0000 C CNN
 F 2 "" H 19000 18350 50  0001 C CNN
@@
 Wire Wire Line
 	22050 18700 22050 18950
+Text GLabel 29950 10700 2    39   Input ~ 0
+SCL_TEENSY
+Text GLabel 29950 10800 2    39   Input ~ 0
+SDA_TEENSY
+NoConn ~ 27650 8200
+NoConn ~ 27650 8300
+NoConn ~ 27650 8500
+NoConn ~ 27650 8600
+NoConn ~ 27650 8700
+NoConn ~ 27650 8800
+NoConn ~ 27650 7600
+NoConn ~ 27650 7500
+NoConn ~ 27650 7400
+NoConn ~ 27650 7300
+Text GLabel 14650 21050 3    50   Input ~ 0
+3.3VBMS
+$Comp
+L bno055:+3.3V #PWR0102
+U 1 1 60605625
+P 14650 20750
+F 0 "#PWR0102" H 14650 20600 50  0001 C CNN
+F 1 "+3.3V" H 14665 20923 50  0000 C CNN
+F 2 "" H 14650 20750 50  0001 C CNN
+F 3 "" H 14650 20750 50  0001 C CNN
+	1    14650 20750
+	1    0    0    -1
+$EndComp
+Wire Wire Line
+	14650 20750 14650 21050
+$Comp
+L power:PWR_FLAG #FLG0101
+U 1 1 6060F62B
+P 2000 19150
+F 0 "#FLG0101" H 2000 19225 50  0001 C CNN
+F 1 "PWR_FLAG" H 2000 19323 50  0000 C CNN
+F 2 "" H 2000 19150 50  0001 C CNN
+F 3 "~" H 2000 19150 50  0001 C CNN
+	1    2000 19150
+	1    0    0    -1
+$EndComp
+Connection ~ 2000 19150
+Wire Wire Line
+	2000 19150 2050 19150
 $EndSCHEMATC

Commit message: change connector, power supply circuit, add buzzer
Parts:
- removed BMS_CONN1, BMS_CONN2: Conn_01x04_Male, Connector_PinHeader_2.54mm:PinHeader_1x04_P2.54mm_Vertical, symbol Connector:Conn_01x04_Male
- removed D1: D, footprints:D_0805_OEM, symbol Device:D
- removed J3: Conn_01x03_Male, Connector_PinHeader_2.54mm:PinHeader_1x03_P2.54mm_Vertical, symbol Connector:Conn_01x03_Male
- added J?: Conn_02x03_Odd_Even, Connector_PinSocket_2.54mm:PinSocket_2x04_P2.54mm_Vertical, symbol Connector_Generic:Conn_02x03_Odd_Even
- added LS?: PKB24SPCH3601-B0, rev2_lib:SPKR_PKB24SPCH3601-B0, symbol rev2:PKB24SPCH3601-B0
Connections:
- net 3.3V_TEENSY is gone; now on net +3V3: U3.15 (3.3V)
- net +3V3: no longer C14.1, U7.7 (OUT)
- net BMS_to_Teensy: now also C14.1, U7.7 (OUT)
- net GND: now also J?.1 (Pin_1), LS?.N
- net MAIN_DEPLOY: now reaches U3.11 (9_PWM_RX2_CS0)
- net MAIN_DEPLOY: now also J?.2 (Pin_2)
- net DROGUE_DEPLOY: now reaches U3.12 (10_PWM_TX2_CS0)
- net DROGUE_DEPLOY: now also J?.4 (Pin_4)
- net BUZZER: now reaches U3.21 (29_PWM_CAN0TX_TOUCH)
- net BUZZER: now also LS?.P
- net BMS_to_sensors renamed 3.3VBMS
- net 3.3VBMS: now also J?.3 (Pin_3)
- net BMS_to_sensors_backup renamed 3.3VBMS_Backup
- net 3.3VBMS_Backup: now also J?.5 (Pin_5)
- no-connect marks 76 -> 72
Other:
- note removed: "3-way switch\nControlled by bridging two of the headers\nDetermines whether the power rail is connected to the\n3.3V pin on the teensy"
- note removed: "power can only flow into the Teensy,\nnot out of the 5V pin"
Changed lines of the file:
@@
 $EndComp
-$Comp
-L power:+3.3V #PWR0114
-U 1 1 6014F363
-P 1750 18900
-F 0 "#PWR0114" H 1750 18750 50  0001 C CNN
-F 1 "+3.3V" H 1765 19073 50  0000 C CNN
-F 2 "" H 1750 18900 50  0001 C CNN
-F 3 "" H 1750 18900 50  0001 C CNN
-	1    1750 18900
-	1    0    0    -1
-$EndComp
-$Comp
-L Connector:Conn_01x03_Male J3
-U 1 1 6017224C
-P 1750 19600
-F 0 "J3" V 1904 19412 50  0000 R CNN
-F 1 "Conn_01x03_Male" V 1813 19412 50  0000 R CNN
-F 2 "Connector_PinHeader_2.54mm:PinHeader_1x03_P2.54mm_Vertical" H 1750 19600 50  0001 C CNN
-F 3 "~" H 1750 19600 50  0001 C CNN
-	1    1750 19600
-	0    -1   -1   0
-$EndComp
-Wire Wire Line
-	1650 19400 1650 19150
-Wire Wire Line
-	1650 19150 1450 19150
-Wire Wire Line
-	1850 19400 1850 19150
-Wire Wire Line
-	1850 19150 2000 19150
-Wire Wire Line
-	1750 19400 1750 18900
-Text Notes 1050 18600 0    50   ~ 0
-3-way switch\nControlled by bridging two of the headers\nDetermines whether the power rail is connected to the\n3.3V pin on the teensy
 $Comp
 L power:+3.3V #PWR0115
@@
 Text GLabel 27650 7900 0    39   Input ~ 0
 3.3V_TEENSY
-Text GLabel 2050 19150 2    39   Input ~ 0
+Text GLabel 10850 19900 3    39   Input ~ 0
 3.3V_TEENSY
-NoConn ~ 1450 19150
 NoConn ~ 18300 12200
 Wire Wire Line
@@
 Text GLabel 29950 10000 2    50   Input ~ 0
 BMS_to_Teensy
-Wire Wire Line
-	9600 19150 9600 19000
-Wire Wire Line
-	9250 19000 9600 19000
-Wire Wire Line
-	9250 18650 9250 19000
-Wire Wire Line
-	8950 18650 8950 19000
-Wire Wire Line
-	8600 19000 8600 19100
-Wire Wire Line
-	8950 19000 8600 19000
-Wire Wire Line
-	8600 19650 8600 19400
-Text GLabel 9150 18800 3    50   Input ~ 0
-BMS_to_sensors
-Text GLabel 9050 18800 3    50   Input ~ 0
-BMS_to_sensors_backup
-Wire Wire Line
-	9050 18650 9050 18800
-Wire Wire Line
-	9150 18650 9150 18800
-Text GLabel 8600 19650 3    50   Input ~ 0
-BMS_to_Teensy
-$Comp
-L power:GND #PWR04
-U 1 1 602C00BA
-P 9600 19150
-F 0 "#PWR04" H 9600 18900 50  0001 C CNN
-F 1 "GND" H 9605 18977 50  0000 C CNN
-F 2 "" H 9600 19150 50  0001 C CNN
-F 3 "" H 9600 19150 50  0001 C CNN
-	1    9600 19150
-	1    0    0    -1
-$EndComp
-$Comp
-L Connector:Conn_01x04_Male BMS_CONN1
-U 1 1 602BDAB1
-P 9150 18450
-F 0 "BMS_CONN1" V 9212 18594 50  0000 L CNN
-F 1 "Conn_01x04_Male" V 9303 18594 50  0000 L CNN
-F 2 "Connector_PinHeader_2.54mm:PinHeader_1x04_P2.54mm_Vertical" H 9150 18450 50  0001 C CNN
-F 3 "~" H 9150 18450 50  0001 C CNN
-	1    9150 18450
-	0    1    1    0
-$EndComp
-Text Notes 6950 19900 0    50   ~ 0
-power can only flow into the Teensy,\nnot out of the 5V pin
-$Comp
-L Device:D D1
-U 1 1 60275618
-P 8600 19250
-F 0 "D1" V 8646 19170 50  0000 R CNN
-F 1 "D" V 8555 19170 50  0000 R CNN
-F 2 "footprints:D_0805_OEM" H 8600 19250 50  0001 C CNN
-F 3 "~" H 8600 19250 50  0001 C CNN
-	1    8600 19250
-	0    -1   -1   0
-$EndComp
-Wire Wire Line
-	6400 19150 6400 19000
-Wire Wire Line
-	6050 19000 6400 19000
-Wire Wire Line
-	6050 18650 6050 19000
-Wire Wire Line
-	5750 18650 5750 19000
-Wire Wire Line
-	5750 19000 5400 19000
-Text GLabel 5950 18800 3    50   Input ~ 0
-BMS_to_sensors
-Text GLabel 5850 18800 3    50   Input ~ 0
-BMS_to_sensors_backup
-Wire Wire Line
-	5850 18650 5850 18800
-Wire Wire Line
-	5950 18650 5950 18800
-$Comp
-L power:GND #PWR015
-U 1 1 6047CFA5
-P 6400 19150
-F 0 "#PWR015" H 6400 18900 50  0001 C CNN
-F 1 "GND" H 6405 18977 50  0000 C CNN
-F 2 "" H 6400 19150 50  0001 C CNN
-F 3 "" H 6400 19150 50  0001 C CNN
-	1    6400 19150
-	1    0    0    -1
-$EndComp
-$Comp
-L Connector:Conn_01x04_Male BMS_CONN2
-U 1 1 6047CFAF
-P 5950 18450
-F 0 "BMS_CONN2" V 6012 18594 50  0000 L CNN
-F 1 "Conn_01x04_Male" V 6103 18594 50  0000 L CNN
-F 2 "Connector_PinHeader_2.54mm:PinHeader_1x04_P2.54mm_Vertical" H 5950 18450 50  0001 C CNN
-F 3 "~" H 5950 18450 50  0001 C CNN
-	1    5950 18450
-	0    1    1    0
-$EndComp
-Wire Wire Line
-	5400 19950 6850 19950
-Wire Wire Line
-	6850 19950 6850 19000
-Wire Wire Line
-	6850 19000 8600 19000
-Wire Wire Line
-	5400 19000 5400 19950
-Connection ~ 8600 19000
 NoConn ~ 27650 9900
 Text Notes 18800 10200 0    250  ~ 0
@@
 	0    1    1    0
 $EndComp
-Text GLabel 13900 18450 1    50   Input ~ 0
-BMS_to_sensors
-Text GLabel 13800 18450 1    50   Input ~ 0
-BMS_to_sensors_backup
 Wire Wire Line
 	13800 18900 13800 18450
@@
 	0    1    1    0
 $EndComp
-Text GLabel 14100 21050 3    50   Input ~ 0
-3.3VBMS
 $Comp
 L preferred_parts:R_475 R5
@@
 NoConn ~ 27650 8200
 NoConn ~ 27650 8300
-NoConn ~ 27650 8500
 NoConn ~ 27650 8600
 NoConn ~ 27650 8700
 NoConn ~ 27650 8800
-NoConn ~ 27650 7600
-NoConn ~ 27650 7500
 NoConn ~ 27650 7400
 NoConn ~ 27650 7300
-Text GLabel 14650 21050 3    50   Input ~ 0
-3.3VBMS
-$Comp
-L bno055:+3.3V #PWR0102
-U 1 1 60605625
-P 14650 20750
-F 0 "#PWR0102" H 14650 20600 50  0001 C CNN
-F 1 "+3.3V" H 14665 20923 50  0000 C CNN
-F 2 "" H 14650 20750 50  0001 C CNN
-F 3 "" H 14650 20750 50  0001 C CNN
-	1    14650 20750
-	1    0    0    -1
-$EndComp
-Wire Wire Line
-	14650 20750 14650 21050
 $Comp
 L power:PWR_FLAG #FLG0101
 U 1 1 6060F62B
-P 2000 19150
-F 0 "#FLG0101" H 2000 19225 50  0001 C CNN
-F 1 "PWR_FLAG" H 2000 19323 50  0000 C CNN
-F 2 "" H 2000 19150 50  0001 C CNN
-F 3 "~" H 2000 19150 50  0001 C CNN
-	1    2000 19150
-	1    0    0    -1
-$EndComp
-Connection ~ 2000 19150
-Wire Wire Line
-	2000 19150 2050 19150
+P 10850 19750
+F 0 "#FLG0101" H 10850 19825 50  0001 C CNN
+F 1 "PWR_FLAG" H 10850 19923 50  0000 C CNN
+F 2 "" H 10850 19750 50  0001 C CNN
+F 3 "~" H 10850 19750 50  0001 C CNN
+	1    10850 19750
+	0    -1   -1   0
+$EndComp
+$Comp
+L Connector_Generic:Conn_02x03_Odd_Even J?
+U 1 1 605F8732
+P 10900 21300
+F 0 "J?" H 10950 21617 50  0000 C CNN
+F 1 "Conn_02x03_Odd_Even" H 10950 21526 50  0000 C CNN
+F 2 "Connector_PinSocket_2.54mm:PinSocket_2x04_P2.54mm_Vertical" H 10900 21300 50  0001 C CNN
+F 3 "~" H 10900 21300 50  0001 C CNN
+	1    10900 21300
+	1    0    0    -1
+$EndComp
+$Comp
+L power:GND #PWR?
+U 1 1 605FA4DA
+P 9800 21200
+F 0 "#PWR?" H 9800 20950 50  0001 C CNN
+F 1 "GND" H 9805 21027 50  0000 C CNN
+F 2 "" H 9800 21200 50  0001 C CNN
+F 3 "" H 9800 21200 50  0001 C CNN
+	1    9800 21200
+	1    0    0    -1
+$EndComp
+Wire Wire Line
+	10700 21200 9800 21200
+Text GLabel 14100 21050 3    50   Input ~ 0
+BMS_to_Teensy
+Text GLabel 10700 21300 0    50   Input ~ 0
+3.3VBMS
+Text GLabel 13900 18450 1    50   Input ~ 0
+3.3VBMS
+Text GLabel 13800 18450 1    50   Input ~ 0
+3.3VBMS_Backup
+Text GLabel 10700 21400 0    50   Input ~ 0
+3.3VBMS_Backup
+$Comp
+L bno055:+3.3V #PWR?
+U 1 1 606115A7
+P 10850 19600
+F 0 "#PWR?" H 10850 19450 50  0001 C CNN
+F 1 "+3.3V" H 10865 19773 50  0000 C CNN
+F 2 "" H 10850 19600 50  0001 C CNN
+F 3 "" H 10850 19600 50  0001 C CNN
+	1    10850 19600
+	1    0    0    -1
+$EndComp
+Wire Wire Line
+	10850 19900 10850 19750
+Wire Wire Line
+	10850 19750 10850 19600
+Connection ~ 10850 19750
+Text GLabel 27650 7500 0    50   Input ~ 0
+MAIN_DEPLOY
+Text GLabel 27650 7600 0    50   Input ~ 0
+DROGUE_DEPLOY
+Text GLabel 11200 21200 2    50   Input ~ 0
+MAIN_DEPLOY
+Text GLabel 11200 21300 2    50   Input ~ 0
+DROGUE_DEPLOY
+$Comp
+L rev2:PKB24SPCH3601-B0 LS?
+U 1 1 6063964C
+P 23550 20100
+F 0 "LS?" H 23654 20191 50  0000 L CNN
+F 1 "PKB24SPCH3601-B0" H 23654 20100 50  0000 L CNN
+F 2 "rev2_lib:SPKR_PKB24SPCH3601-B0" H 23654 20009 50  0000 L CNN
+F 3 "https://www.murata.com/~/media/webrenewal/support/library/catalog/products/sound/p37e.ashx?la=en-us#page=18" H 23550 20100 50  0001 L BNN
+F 4 "Murata Electronics" H 23550 20100 50  0001 L BNN "MANUFACTURER"
+F 5 "10.0 mm" H 23550 20100 50  0001 L BNN "MAXIMUM_PACKAGE_HEIGHT"
+F 6 "IPC-7351B" H 23550 20100 50  0001 L BNN "STANDARD"
+F 7 "March 24, 2017" H 23550 20100 50  0001 L BNN "PARTREV"
+	1    23550 20100
+	1    0    0    -1
+$EndComp
+Text GLabel 23550 19550 1    50   Input ~ 0
+BUZZER
+$Comp
+L power:GND #PWR?
+U 1 1 6063B873
+P 23550 20650
+F 0 "#PWR?" H 23550 20400 50  0001 C CNN
+F 1 "GND" H 23555 20477 50  0000 C CNN
+F 2 "" H 23550 20650 50  0001 C CNN
+F 3 "" H 23550 20650 50  0001 C CNN
+	1    23550 20650
+	1    0    0    -1
+$EndComp
+Wire Wire Line
+	23550 19550 23550 19900
+Wire Wire Line
+	23550 20300 23550 20650
+Text GLabel 27650 8500 0    50   Input ~ 0
+BUZZER
 $EndSCHEMATC

Commit message: start layout
Parts:
- J3: renamed from J?; footprint Connector_PinSocket_2.54mm:PinSocket_2x04_P2.54mm_Vertical -> Connector_PinHeader_2.54mm:PinHeader_2x03_P2.54mm_Vertical
- gave numbers to parts that had none: 1
Changed lines of the file:
@@
 $EndComp
 $Comp
-L Connector_Generic:Conn_02x03_Odd_Even J?
+L Connector_Generic:Conn_02x03_Odd_Even J3
 U 1 1 605F8732
 P 10900 21300
-F 0 "J?" H 10950 21617 50  0000 C CNN
+F 0 "J3" H 10950 21617 50  0000 C CNN
 F 1 "Conn_02x03_Odd_Even" H 10950 21526 50  0000 C CNN
-F 2 "Connector_PinSocket_2.54mm:PinSocket_2x04_P2.54mm_Vertical" H 10900 21300 50  0001 C CNN
+F 2 "Connector_PinHeader_2.54mm:PinHeader_2x03_P2.54mm_Vertical" H 10900 21300 50  0001 C CNN
 F 3 "~" H 10900 21300 50  0001 C CNN
 	1    10900 21300
@@
 $EndComp
 $Comp
-L power:GND #PWR?
+L power:GND #PWR0102
 U 1 1 605FA4DA
 P 9800 21200
-F 0 "#PWR?" H 9800 20950 50  0001 C CNN
+F 0 "#PWR0102" H 9800 20950 50  0001 C CNN
 F 1 "GND" H 9805 21027 50  0000 C CNN
 F 2 "" H 9800 21200 50  0001 C CNN
@@
 3.3VBMS_Backup
 $Comp
-L bno055:+3.3V #PWR?
+L bno055:+3.3V #PWR0105
 U 1 1 606115A7
 P 10850 19600
-F 0 "#PWR?" H 10850 19450 50  0001 C CNN
+F 0 "#PWR0105" H 10850 19450 50  0001 C CNN
 F 1 "+3.3V" H 10865 19773 50  0000 C CNN
 F 2 "" H 10850 19600 50  0001 C CNN
@@
 DROGUE_DEPLOY
 $Comp
-L rev2:PKB24SPCH3601-B0 LS?
+L rev2:PKB24SPCH3601-B0 LS1
 U 1 1 6063964C
 P 23550 20100
-F 0 "LS?" H 23654 20191 50  0000 L CNN
+F 0 "LS1" H 23654 20191 50  0000 L CNN
 F 1 "PKB24SPCH3601-B0" H 23654 20100 50  0000 L CNN
 F 2 "rev2_lib:SPKR_PKB24SPCH3601-B0" H 23654 20009 50  0000 L CNN
@@
 BUZZER
 $Comp
-L power:GND #PWR?
+L power:GND #PWR0109
 U 1 1 6063B873
 P 23550 20650
-F 0 "#PWR?" H 23550 20400 50  0001 C CNN
+F 0 "#PWR0109" H 23550 20400 50  0001 C CNN
 F 1 "GND" H 23555 20477 50  0000 C CNN
 F 2 "" H 23550 20650 50  0001 C CNN
