File: hardware/rev2/rev2.sch (KiCad schematic (older format))
At the start: 34 parts, among them J1 Conn_01x09_Female, J2 RFM9X_header, J3 Conn_02x03_Odd_Even, U2 MPL3115A2, U3 Teensy3.6, U5 ADXL345BCCZ, U7 TPS2113ADRBR

Commit message: change silkscreen
Parts:
- D2, D3, D4, D5, D6, D7: footprint KingbrightLED:AA3528LSECKT-J4 -> rev2_lib:AA3528LSECKT-J4
Changed lines of the file:
@@
 F 0 "D3" V 24789 19632 50  0000 R CNN
 F 1 "LED" V 24698 19632 50  0000 R CNN
-F 2 "KingbrightLED:AA3528LSECKT-J4" H 24750 19750 50  0001 C CNN
+F 2 "rev2_lib:AA3528LSECKT-J4" H 24750 19750 50  0001 C CNN
 F 3 "~" H 24750 19750 50  0001 C CNN
 	1    24750 19750
@@
 F 0 "D2" V 22647 19630 50  0000 L CNN
 F 1 "LED" V 22738 19630 50  0000 L CNN
-F 2 "KingbrightLED:AA3528LSECKT-J4" H 22700 19550 50  0001 C CNN
+F 2 "rev2_lib:AA3528LSECKT-J4" H 22700 19550 50  0001 C CNN
 F 3 "~" H 22700 19550 50  0001 C CNN
 	1    22700 19550
@@
 F 0 "D4" V 27247 16630 50  0000 L CNN
 F 1 "LED" V 27338 16630 50  0000 L CNN
-F 2 "KingbrightLED:AA3528LSECKT-J4" H 27300 16550 50  0001 C CNN
+F 2 "rev2_lib:AA3528LSECKT-J4" H 27300 16550 50  0001 C CNN
 F 3 "~" H 27300 16550 50  0001 C CNN
 	1    27300 16550
@@
 F 0 "D5" V 27997 16630 50  0000 L CNN
 F 1 "LED" V 28088 16630 50  0000 L CNN
-F 2 "KingbrightLED:AA3528LSECKT-J4" H 28050 16550 50  0001 C CNN
+F 2 "rev2_lib:AA3528LSECKT-J4" H 28050 16550 50  0001 C CNN
 F 3 "~" H 28050 16550 50  0001 C CNN
 	1    28050 16550
@@
 F 0 "D6" V 28747 16630 50  0000 L CNN
 F 1 "LED" V 28838 16630 50  0000 L CNN
-F 2 "KingbrightLED:AA3528LSECKT-J4" H 28800 16550 50  0001 C CNN
+F 2 "rev2_lib:AA3528LSECKT-J4" H 28800 16550 50  0001 C CNN
 F 3 "~" H 28800 16550 50  0001 C CNN
 	1    28800 16550
@@
 F 0 "D7" V 29497 16630 50  0000 L CNN
 F 1 "LED" V 29588 16630 50  0000 L CNN
-F 2 "KingbrightLED:AA3528LSECKT-J4" H 29550 16550 50  0001 C CNN
+F 2 "rev2_lib:AA3528LSECKT-J4" H 29550 16550 50  0001 C CNN
 F 3 "~" H 29550 16550 50  0001 C CNN
 	1    29550 16550

Commit message: create footprint for Rev2 Molex Connector
Parts:
- J3: footprint Connector_PinHeader_2.54mm:PinHeader_2x03_P2.54mm_Vertical -> footprints:Molex_Nano-Fit_105312-1106; symbol Connector_Generic:Conn_02x03_Odd_Even -> Connector_Generic:Conn_02x03_Top_Bottom
Connections:
- net 3.3VBMS: now also J3.4 (Pin_4); no longer J3.2 (Pin_2)
- net 3.3VBMS_Backup: now also J3.5 (Pin_5); no longer J3.4 (Pin_4)
- net DROGUE_DEPLOY: now also J3.3 (Pin_3); no longer J3.5 (Pin_5)
Changed lines of the file:
@@
 $EndComp
 $Comp
-L Connector_Generic:Conn_02x03_Odd_Even J3
+L Connector_Generic:Conn_02x03_Top_Bottom J3
 U 1 1 605F8732
 P 2600 21400
 F 0 "J3" H 2650 21717 50  0000 C CNN
 F 1 "Conn_02x03_Odd_Even" H 2650 21626 50  0000 C CNN
-F 2 "Connector_PinHeader_2.54mm:PinHeader_2x03_P2.54mm_Vertical" H 2600 21400 50  0001 C CNN
-F 3 "~" H 2600 21400 50  0001 C CNN
+F 2 "footprints:Molex_Nano-Fit_105312-1106" H 2600 21400 50  0001 C CNN
+F 3 "https://www.molex.com/pdm_docs/sd/1053121104_sd.pdf" H 2600 21400 50  0001 C CNN
 	1    2600 21400
 	1    0    0    -1
