File: hardware/REV2_SPRING_2022/REV2_SPRING_2022.kicad_pcb (KiCad board)
At the start: 2 copper layers, 108 x 304.8 mm, 52 parts, among them J101 Screw_Terminal_01x02, J102 Screw_Terminal_01x02, J103 Conn_01x02_Female, J104 Screw_Terminal_01x02, J105 Conn_01x02_Female, J107 Screw_Terminal_01x02, J109 Conn_01x02_Female, J110 Conn_01x02_Female, Q101 Q_NMOS_GDS, Q102 Q_NMOS_GDS, U1 Teensy3.6_All_Pins, U2 PA16165_Breakout, U201 TPS2113ADRBR, U3 MPL3115A2_Breakout, U301 TPS2113ADRBR, U4 BNO055_Breakout, U5 RFM69HCW_Breakout

Commit message: finish routing
Routing:
- net /BAT2: track 38.4 -> 164.2 mm, vias 0 -> 2
- net /BAT1: track 48.5 -> 85.6 mm
Changed lines of the file:
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@@
     (thickness 1.6)
     (drawings 26)
-    (tracks 323)
+    (tracks 348)
     (zones 0)
     (modules 52)
@@
   )
   (setup
-    (last_trace_width 1.524)
+    (last_trace_width 0.4318)
     (user_trace_width 0.4318)
     (user_trace_width 0.762)
@@
   (segment (start 132.5 164.5) (end 135.4265 167.4265) (width 0.4318) (layer F.Cu) (net 35))
   (via (at 123.499972 167.25) (size 0.8) (drill 0.4) (layers F.Cu B.Cu) (net 35))
-  (segment (start 129.75 167.25) (end 123.499972 167.25) (width 0.4318) (layer B.Cu) (net 35))
   (segment (start 116.7075 167.323) (end 123.426972 167.323) (width 0.4318) (layer F.Cu) (net 35))
   (segment (start 123.426972 167.323) (end 123.499972 167.25) (width 0.4318) (layer F.Cu) (net 35))
-  (segment (start 132.5 164.5) (end 129.75 167.25) (width 0.4318) (layer B.Cu) (net 35))
+  (segment (start 126.5 167.25) (end 123.499972 167.25) (width 0.4318) (layer B.Cu) (net 35))
+  (segment (start 129.25 164.5) (end 126.5 167.25) (width 0.4318) (layer B.Cu) (net 35))
+  (segment (start 132.5 164.5) (end 129.25 164.5) (width 0.4318) (layer B.Cu) (net 35))
   (segment (start 107 150) (end 96.5 160.5) (width 0.25) (layer B.Cu) (net 36))
   (segment (start 107 141.8) (end 107 150) (width 0.25) (layer B.Cu) (net 36))
@@
   (segment (start 131.04 171.6515) (end 129.225 173.4665) (width 0.4318) (layer F.Cu) (net 121) (status 20))
   (segment (start 131.04 168.7265) (end 131.04 171.6515) (width 0.4318) (layer F.Cu) (net 121) (status 10))
-  (segment (start 135.409 175.5) (end 140.062 170.847) (width 0.4318) (layer F.Cu) (net 121) (status 20))
-  (segment (start 131.25 175.5) (end 135.409 175.5) (width 0.4318) (layer F.Cu) (net 121))
   (segment (start 129.225 173.475) (end 131.25 175.5) (width 0.4318) (layer F.Cu) (net 121) (status 10))
   (segment (start 129.225 173.4665) (end 129.225 173.475) (width 0.4318) (layer F.Cu) (net 121) (status 30))
   (segment (start 110.9825 170.913) (end 108.5325 173.363) (width 0.4318) (layer F.Cu) (net 121) (status 20))
-  (segment (start 110.9825 168.623) (end 110.9825 170.913) (width 0.4318) (layer F.Cu) (net 121) (status 10))
   (segment (start 108.5325 173.363) (end 108.613 173.363) (width 0.4318) (layer F.Cu) (net 121) (status 30))
-  (segment (start 110.75 175.5) (end 131.25 175.5) (width 0.4318) (layer F.Cu) (net 121))
   (segment (start 108.613 173.363) (end 110.75 175.5) (width 0.4318) (layer F.Cu) (net 121) (status 10))
+  (segment (start 155.555 186.305) (end 155.555 188.72) (width 0.4318) (layer F.Cu) (net 121))
+  (segment (start 135.409 175.5) (end 144.75 175.5) (width 0.4318) (layer F.Cu) (net 121))
+  (segment (start 144.75 175.5) (end 155.555 186.305) (width 0.4318) (layer F.Cu) (net 121))
+  (segment (start 140.097 170.847) (end 144.75 175.5) (width 0.4318) (layer F.Cu) (net 121))
+  (segment (start 140.062 170.847) (end 140.097 170.847) (width 0.4318) (layer F.Cu) (net 121))
+  (segment (start 110.75 175.5) (end 113 175.5) (width 0.4318) (layer F.Cu) (net 121))
+  (segment (start 113 175.5) (end 131.25 175.5) (width 0.4318) (layer F.Cu) (net 121))
+  (segment (start 110.9825 173.4825) (end 110.9825 168.623) (width 0.4318) (layer F.Cu) (net 121))
+  (segment (start 113 175.5) (end 110.9825 173.4825) (width 0.4318) (layer F.Cu) (net 121))
+  (segment (start 131.25 175.5) (end 133 175.5) (width 0.4318) (layer F.Cu) (net 121))
+  (segment (start 133 175.5) (end 135.409 175.5) (width 0.4318) (layer F.Cu) (net 121))
+  (segment (start 131.04 173.54) (end 131.04 171.6515) (width 0.4318) (layer F.Cu) (net 121))
+  (segment (start 133 175.5) (end 131.04 173.54) (width 0.4318) (layer F.Cu) (net 121))
   (segment (start 131.04 167.4265) (end 130.1765 167.4265) (width 0.4318) (layer F.Cu) (net 122) (status 10))
   (segment (start 129.225 166.475) (end 129.225 162.0365) (width 0.4318) (layer F.Cu) (net 122) (status 20))
@@
   (segment (start 108.511 165.761) (end 108.511 162.7165) (width 0.4318) (layer F.Cu) (net 122) (status 20))
   (segment (start 110.073 167.323) (end 108.511 165.761) (width 0.4318) (layer F.Cu) (net 122))
-  (segment (start 129.225 162.0365) (end 154.7865 162.0365) (width 0.4318) (layer F.Cu) (net 122) (status 10))
+  (segment (start 129.225 162.0365) (end 147.5365 162.0365) (width 0.4318) (layer F.Cu) (net 122))
+  (segment (start 163.5 202.365) (end 155.555 210.31) (width 0.4318) (layer F.Cu) (net 122))
+  (segment (start 163.5 178) (end 163.5 202.365) (width 0.4318) (layer F.Cu) (net 122))
+  (segment (start 108.511 165.761) (end 107.25 164.5) (width 0.4318) (layer F.Cu) (net 122))
+  (via (at 105.75 164.5) (size 1.016) (drill 0.635) (layers F.Cu B.Cu) (net 122))
+  (segment (start 107.25 164.5) (end 105.75 164.5) (width 0.4318) (layer F.Cu) (net 122))
+  (via (at 155.5 176.25) (size 1.016) (drill 0.635) (layers F.Cu B.Cu) (net 122))
+  (segment (start 161.75 176.25) (end 163.125 177.625) (width 0.4318) (layer F.Cu) (net 122))
+  (segment (start 155.5 176.25) (end 161.75 176.25) (width 0.4318) (layer F.Cu) (net 122))
+  (segment (start 163.125 177.625) (end 163.5 178) (width 0.4318) (layer F.Cu) (net 122))
+  (segment (start 147.5365 162.0365) (end 163.125 177.625) (width 0.4318) (layer F.Cu) (net 122))
+  (segment (start 108.25 176.25) (end 155.5 176.25) (width 0.4318) (layer B.Cu) (net 122))
+  (segment (start 102.75 170.75) (end 108.25 176.25) (width 0.4318) (layer B.Cu) (net 122))
+  (segment (start 102.75 166) (end 102.75 170.75) (width 0.4318) (layer B.Cu) (net 122))
+  (segment (start 104.25 164.5) (end 102.75 166) (width 0.4318) (layer B.Cu) (net 122))
+  (segment (start 105.75 164.5) (end 104.25 164.5) (width 0.4318) (layer B.Cu) (net 122))
   (segment (start 109.0645 167.973) (end 108.5375 168.5) (width 0.4318) (layer F.Cu) (net 123) (status 30))
   (segment (start 110.9825 167.973) (end 109.0645 167.973) (width 0.4318) (layer F.Cu) (net 123) (status 30))
